Commit message: aggiunto jac ma non serve perché sono stupido mannaggia

File: truck_description/urdf/truck.xacro (robot description, xacro)
@@ -2,4 +2,10 @@
 <robot name="truck" xmlns:xacro="http://www.ros.org/wiki/xacro">
 <xacro:include filename="$(find truck_description)/urdf/materials.xacro" />
+<link name="base_wrench_sensor"/>
+<joint name="base_wrench_sensor_joint" type="fixed">
+  <parent link="base_link"/>
+  <child link="base_wrench_sensor"/>
+  <origin xyz="0 0 0" rpy="0 0 0"/>
+</joint>
 <link name="base_link">
   <inertial>

Commit message: Gazebo and model coexist

File: truck_description/urdf/truck.xacro (robot description, xacro)
@@ -2,10 +2,4 @@
 <robot name="truck" xmlns:xacro="http://www.ros.org/wiki/xacro">
 <xacro:include filename="$(find truck_description)/urdf/materials.xacro" />
-<link name="base_wrench_sensor"/>
-<joint name="base_wrench_sensor_joint" type="fixed">
-  <parent link="base_link"/>
-  <child link="base_wrench_sensor"/>
-  <origin xyz="0 0 0" rpy="0 0 0"/>
-</joint>
 <link name="base_link">
   <inertial>
@@ -406,5 +400,5 @@
     <origin xyz="0 0 0" rpy="0 0 0"/>
     <geometry>
-      <sphere radius="0.15"/>
+      <sphere radius="0.00015"/>
     </geometry>
   </collision>
@@ -424,5 +418,5 @@
   <parent link="base_link"/>
   <child link="imu_link"/>
-  <origin xyz="-2.317907 0.060311 2.084352" rpy="0 0 0"/>
+  <origin xyz="-2.317907 0.060311 2.084352" rpy="0 0 3.14"/>
 </joint>
 </robot>
