Commit message: messo anche gazebo e sto vedendo l'imu di mujoco, che da numeri diversi da vx*wz

File: truck_control/urdf/truck_control.xacro (robot description, xacro)
@@ -3,8 +3,12 @@
 <xacro:arg name="driven_wheels" default="8"/>
 <xacro:arg name="steering_limit" default="${35 * pi / 180}"/>
+<xacro:arg name="gz_sim" default="false" />
+<!-- 2. Convert arguments to xacro properties for evaluation -->
+<xacro:property name="gz_sim" value="$(arg gz_sim)" />
 <xacro:include filename="$(find truck_control)/urdf/truck8x$(arg driven_wheels)_control.ros2control" />
-<!-- That is the way gz call the control manager. Do it by launch file instead in this setting
-<xacro:include filename="$(find truck_control)/urdf/truck_control.gazebo" />
- -->
+<!-- That is the way gz call the control manager. Do it by launch file instead in this setting -->
+<xacro:if value="${gz_sim}">
+  <xacro:include filename="$(find truck_control)/urdf/truck_control.gazebo" />
+</xacro:if>
 <!--Extension of base xacro with fictitious link and fixed joint in order to compute odometry of application point-->
 <xacro:arg name="app_point_offset" default="0.0"/>

File: truck_description/urdf/piramide_truck.xacro (robot description, xacro)
@@ -5,4 +5,5 @@
   <xacro:arg name="app_point_offset" default="0.0"/>
   <xacro:arg name="steering_limit" default="${35 * pi / 180}"/>
+  <xacro:arg name="gz_sim" default="false" />
   <xacro:include filename="$(find truck_description)/urdf/truck.xacro" />
   <xacro:if value="${'$(arg control_mode)' == 'control'}">

Commit message: csv

File: truck_control/urdf/truck_control.xacro (robot description, xacro)
@@ -3,7 +3,14 @@
 <xacro:arg name="driven_wheels" default="8"/>
 <xacro:arg name="steering_limit" default="${35 * pi / 180}"/>
+<!-- argument to place base_footprint at the same height as the wheels' center. Useful for observer -->
+<xacro:arg name="footprint_z_offset" default="0.602025" />
+<!-- argument to specify whether a Gazebo or MuJoCo simulation shall be launched -->
+<xacro:arg name="sim_type" default="gazebo" />
 <xacro:include filename="$(find truck_control)/urdf/truck8x$(arg driven_wheels)_control.ros2control" />
-<xacro:include filename="$(find truck_control)/urdf/truck_control.gazebo" />
-<!--Extension of base xacro with fictitious link and fixed joint in order to compute odometry of application point-->
+<!-- if sim_type is 'gazebo', include file truck_control.gazebo containing Gazebo configuration of sensors, odometry, controllers, physics, etc. -->
+<xacro:if value="${'$(arg sim_type)' == 'gazebo'}">
+  <xacro:include filename="$(find truck_control)/urdf/truck_control.gazebo" />
+</xacro:if>
+<!--Extension of base xacro with fictitious link and fixed joint in order to compute odometry at the chosen application point-->
 <xacro:arg name="app_point_offset" default="0.0"/>
 <xacro:arg name="rear_centerline_pos" default="2.6815"/>
@@ -16,6 +23,6 @@
 <joint name="base_joint" type="fixed">
   <parent link="base_footprint"/>
-  <child link="base_link"/>
-  <origin xyz="${$(arg rear_centerline_pos) - $(arg app_point_offset)} 0 0" rpy="0 0 ${pi}"/>
+  <child link="${base_link_name}"/>
+  <origin xyz="${$(arg rear_centerline_pos) - $(arg app_point_offset)} 0 ${$(arg footprint_z_offset)}" rpy="0 0 ${pi}"/>
 </joint>
 </robot>
